File: PC-Power-Control.kicad_sch (KiCad schematic)
At the start: 9 parts, among them J1 Conn_02x06_Odd_Even

Commit message: update
Parts:
- renumbered POWER1 to J1, J1 to J2, RESET-RESISTOR1 to R1, POWER-RESISTOR1 to R2, LED-RESISTOR1 to R3, RESET-SWITCH1 to U1, POWER-SWITCH1 to U2, LED-SWITCH1 to U3
Changed lines of the file:
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@@
   (symbol (lib_id "Device:R") (at 224.79 60.96 90) (unit 1)
     (in_bom yes) (on_board yes) (dnp no) (fields_autoplaced)
-    (property "Reference" "LED-RESISTOR1" (at 224.79 54.61 90)
+    (property "Reference" "R3" (at 224.79 54.61 90)
       (effects (font (size 1.27 1.27)))
     )
@@
       (project "PC-Power-Control"
         (path "/b176fc4e-680d-43fa-882a-ac6582b0a032"
-          (reference "LED-RESISTOR1") (unit 1)
+          (reference "R3") (unit 1)
         )
       )
@@
   (symbol (lib_id "Isolator:EL817") (at 124.46 43.18 0) (unit 1)
     (in_bom yes) (on_board yes) (dnp no) (fields_autoplaced)
-    (property "Reference" "RESET-SWITCH1" (at 124.46 34.29 0)
+    (property "Reference" "U1" (at 124.46 34.29 0)
       (effects (font (size 1.27 1.27)))
     )
@@
       (project "PC-Power-Control"
         (path "/b176fc4e-680d-43fa-882a-ac6582b0a032"
-          (reference "RESET-SWITCH1") (unit 1)
+          (reference "U1") (unit 1)
         )
       )
@@
   (symbol (lib_id "Connector_Generic:Conn_01x02") (at 83.82 124.46 0) (unit 1)
     (in_bom yes) (on_board yes) (dnp no) (fields_autoplaced)
-    (property "Reference" "POWER1" (at 86.36 124.46 0)
+    (property "Reference" "J1" (at 86.36 124.46 0)
       (effects (font (size 1.27 1.27)) (justify left))
     )
@@
       (project "PC-Power-Control"
         (path "/b176fc4e-680d-43fa-882a-ac6582b0a032"
-          (reference "POWER1") (unit 1)
+          (reference "J1") (unit 1)
         )
       )
@@
   (symbol (lib_id "Connector_Generic:Conn_02x06_Odd_Even") (at 149.86 127 0) (unit 1)
     (in_bom yes) (on_board yes) (dnp no) (fields_autoplaced)
-    (property "Reference" "J1" (at 151.13 115.57 0)
+    (property "Reference" "J2" (at 151.13 115.57 0)
       (effects (font (size 1.27 1.27)))
     )
@@
       (project "PC-Power-Control"
         (path "/b176fc4e-680d-43fa-882a-ac6582b0a032"
-          (reference "J1") (unit 1)
+          (reference "J2") (unit 1)
         )
       )
@@
   (symbol (lib_id "Device:R") (at 172.72 60.96 90) (unit 1)
     (in_bom yes) (on_board yes) (dnp no) (fields_autoplaced)
-    (property "Reference" "POWER-RESISTOR1" (at 172.72 54.61 90)
+    (property "Reference" "R2" (at 172.72 54.61 90)
       (effects (font (size 1.27 1.27)))
     )
@@
       (project "PC-Power-Control"
         (path "/b176fc4e-680d-43fa-882a-ac6582b0a032"
-          (reference "POWER-RESISTOR1") (unit 1)
+          (reference "R2") (unit 1)
         )
       )
@@
   (symbol (lib_id "Isolator:EL817") (at 172.72 43.18 0) (unit 1)
     (in_bom yes) (on_board yes) (dnp no) (fields_autoplaced)
-    (property "Reference" "POWER-SWITCH1" (at 172.72 34.29 0)
+    (property "Reference" "U2" (at 172.72 34.29 0)
       (effects (font (size 1.27 1.27)))
     )
@@
       (project "PC-Power-Control"
         (path "/b176fc4e-680d-43fa-882a-ac6582b0a032"
-          (reference "POWER-SWITCH1") (unit 1)
+          (reference "U2") (unit 1)
         )
       )
@@
   (symbol (lib_id "Isolator:EL817") (at 226.06 43.18 0) (unit 1)
     (in_bom yes) (on_board yes) (dnp no) (fields_autoplaced)
-    (property "Reference" "LED-SWITCH1" (at 226.06 34.29 0)
+    (property "Reference" "U3" (at 226.06 34.29 0)
       (effects (font (size 1.27 1.27)))
     )
@@
       (project "PC-Power-Control"
         (path "/b176fc4e-680d-43fa-882a-ac6582b0a032"
-          (reference "LED-SWITCH1") (unit 1)
+          (reference "U3") (unit 1)
         )
       )
@@
   (symbol (lib_id "Device:R") (at 124.46 60.96 90) (unit 1)
     (in_bom yes) (on_board yes) (dnp no) (fields_autoplaced)
-    (property "Reference" "RESET-RESISTOR1" (at 124.46 54.61 90)
+    (property "Reference" "R1" (at 124.46 54.61 90)
       (effects (font (size 1.27 1.27)))
     )
@@
       (project "PC-Power-Control"
         (path "/b176fc4e-680d-43fa-882a-ac6582b0a032"
-          (reference "RESET-RESISTOR1") (unit 1)
-        )
-      )
+          (reference "R1") (unit 1)
+        )
+      )
